File: keyboard.kicad_pcb (KiCad board)
At the start: 2 copper layers, 285 x 94.6 mm, 171 parts, among them J1 USBMINI_B05, K1 DownloadKey, P1 SWD, U1 E73-2G4M04S1D, U2 CH552T, U3 TP4057, U4 XC6206P30

Commit message: 修正原理图两处错误，添加Bootloader按钮
版本设定为B2版本，修正了原理图的两处错误，添加了Bootloadler按钮便于进入DFU刷机模式。
Parts:
- removed LED6: LED, custom:MX1A-led
- removed RL6: 300, 0805:0805R
- removed SJ6: SOLDER_JUMPER, custom:2_Pin_Jumper
- added SW1: Bootloader Button, dtsm:Switch, B.Cu at (91.4, 112.8)
- turned D101 to 90 degrees
Connections:
- D101 pad 1: Net-(D101-Pad1) -> VCC
- D101 pad 2: VCC -> Net-(D101-Pad2)
- R1 pad 2: UD- -> UD+
- U1 pad 20: /led5 -> /DFU
- U2 pad 14: UD- -> UD+
- U2 pad 15: UD+ -> UD-
- U3 pad 4: Net-(D101-Pad1) -> Net-(D101-Pad2)
Routing:
- net /DFU: track 0.00 -> 122.1 mm, vias 0 -> 2
- net /led5: track 91.9 -> 0.00 mm, vias 3 -> 0
- net UD+: track 110.2 -> 120.9 mm
- net UD-: track 120.9 -> 112.1 mm, vias 0 -> 2
- net Net-(LED6-Pad2): track 7.47 -> 0.00 mm
- net /col4: track 112.8 -> 118.9 mm
- net /col6: track 113.7 -> 119.0 mm
- net /col2: track 164.1 -> 169.3 mm
- net /col12: track 190.7 -> 195.9 mm
- net /col7: track 92.9 -> 97.9 mm
- net Net-(D101-Pad2): track 0.00 -> 4.01 mm
- net Net-(D101-Pad1): track 4.01 -> 0.00 mm
- net /col11: track 173.5 -> 176.5 mm
- net /row4: track 354.4 -> 351.5 mm
- net /row3: track 350.7 -> 348.0 mm
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- added copper zone on F.Cu, net (none)
Other:
- board text added: "DATE : 20190301"
- board text added: "GT BLE60"
- board text added: "GT BLE60 Rev.B2 ©2019 Genosoft"
- board text removed: "DATE : 20190210"
- board text removed: "GT BLE60 Rev.B ©2019 Genosoft"

Commit message: 添加SWD接口丝印
Parts:
- moved G*** 3.78 mm to (239.1, 155.7)
- moved LOGO1 3.78 mm to (232.3, 146.8)
- moved LOGO2 3.78 mm to (219.7, 147.0)
Other:
- board text added: "3.3V"
- board text added: "CLK"
- board text added: "GND"
- board text added: "SWI"
Changed lines of the file:
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@@
   (general
     (thickness 1.6)
-    (drawings 104)
+    (drawings 108)
     (tracks 2095)
     (zones 0)
@@
     (36 B.SilkS user)
     (37 F.SilkS user)
-    (38 B.Mask user hide)
+    (38 B.Mask user)
     (39 F.Mask user)
     (40 Dwgs.User user hide)
@@
   )
   (module logos:GTBLE60 (layer B.Cu)
-    (at 228.525 146.955 180)
+    (at 232.305 146.845 180)
     (fp_text reference LOGO1 (at 0.33 4.28 180) (layer B.SilkS) hide
       (effects (font (size 1.524 1.524) (thickness 0.3)) (justify mirror))
@@
     (descr "Through hole straight socket strip, 1x04, 2.54mm pitch, single row (from Kicad 4.0.7), script generated")
     (tags "Through hole socket strip THT 1x04 2.54mm single row")
-    (fp_text reference P1 (at -2.59 -4.08 180) (layer B.SilkS)
+    (fp_text reference P1 (at -2.85 2.04 180) (layer B.SilkS)
       (effects (font (size 1 1) (thickness 0.15)) (justify mirror))
     )
@@
   )
   (module logos:Bluetooth (layer B.Cu)
-    (at 215.95 147.155 180)
+    (at 219.73 147.045 180)
     (fp_text reference LOGO2 (at 0.17 -4.15 180) (layer B.CrtYd) hide
       (effects (font (size 1.524 1.524) (thickness 0.3)) (justify mirror))
@@
   )
   (module logos:keyboard (layer B.Cu)
-    (at 235.3 155.78 180)
+    (at 239.08 155.67 180)
     (fp_text reference G*** (at 0 0 180) (layer B.CrtYd) hide
       (effects (font (size 1.524 1.524) (thickness 0.3)) (justify mirror))
@@
     )
   )
+  (gr_text "GND\n" (at 209.22 153.39) (layer B.Mask)
+    (effects (font (size 1 1) (thickness 0.18)) (justify mirror))
+  )
+  (gr_text CLK (at 209.34 150.84) (layer B.Mask)
+    (effects (font (size 1 1) (thickness 0.18)) (justify mirror))
+  )
+  (gr_text SWI (at 209.3 148.19) (layer B.Mask)
+    (effects (font (size 1 1) (thickness 0.18)) (justify mirror))
+  )
+  (gr_text "3.3V\n" (at 209.26 145.85) (layer B.Mask)
+    (effects (font (size 1 1) (thickness 0.18)) (justify mirror))
+  )
   (gr_text "DATE : 20190301" (at 228.2 154.66) (layer F.SilkS)
     (effects (font (size 1.524 1.016) (thickness 0.254)))
@@
     (effects (font (size 4.064 3.048) (thickness 0.3048)))
   )
-  (gr_text "DATE : 20190301" (at 223.475 156.105) (layer B.Mask)
+  (gr_text "DATE : 20190301" (at 227.255 155.995) (layer B.Mask)
     (effects (font (size 1.3 1.3) (thickness 0.3)) (justify mirror))
   )
@@
     (arrow2b (pts (xy 31.21 92.52) (xy 30.62358 91.393497)))
   )
-  (gr_text "GT BLE60 Rev.B2 ©2019 Genosoft" (at 227.14 152.36) (layer B.Mask)
+  (gr_text "GT BLE60 Rev.B2 ©2019 Genosoft" (at 230.92 152.25) (layer B.Mask)
     (effects (font (size 1.3 1.3) (thickness 0.25)) (justify mirror))
   )
